File: ext_pcb.brd (EAGLE design)
At the start: 100 x 100 mm, 38 parts, among them CN10 MCV_05/4-G-2,5V, CN11 MCV_05/4-G-2,5V, CN12 MCV_05/4-G-2,5V, CN13 MCV_05/4-G-2,5V, CN15 MCV_05/2-G-2,5V, CN16 MCV_05/2-G-2,5V, CN17 MCV_05/2-G-2,5V, CN2 53047-08, CN3 53047-06, CN4 MCV_05/4-G-2,5V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

Commit message: First Draft PCB Design
Parts:
- moved CN17 0.25 mm to (23.2, 95.1)
Routing:
- net VCC: track 316.1 -> 319.8 mm
- net CN3_GND: track 0.00 -> 1.25 mm
- net GND: track 13.3 -> 14.0 mm
- removed copper zone on layer 16, net N$9
Other:
- board text added: "3.3V"
- board text added: "5V"
- board text added: "Boiko, Chehadeh, Alansari, Ayyad, Alrheis"
- board text added: "GND"
- board text removed: "Boiko, Chehadeh"

Commit message: Final Draft
Routing:
- net N$12: track 18.8 -> 20.1 mm
Changed lines of the file:
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@@
 <text x="10.5" y="75.97" size="1.778" layer="21" rot="R90">Boost converter</text>
 <text x="86.085" y="74.825" size="1.778" layer="21" rot="R90">Bluetooth Module</text>
-<text x="29.465" y="41.885" size="3.81" layer="21">MultiWii Board</text>
+<text x="23.935" y="41.345" size="3.81" layer="21">MultiWii Board</text>
 <wire x1="0" y1="0" x2="0" y2="100" width="0.2032" layer="20"/>
 <wire x1="0" y1="100" x2="100" y2="100" width="0.2032" layer="20"/>
@@
 <text x="7.71" y="47.46" size="1.016" layer="21" rot="R90">5V</text>
 <text x="26.33" y="97.69" size="0.508" layer="21" rot="R180">3.3V</text>
+<wire x1="2.87" y1="70.89" x2="2.79" y2="70.89" width="0.254" layer="21"/>
+<wire x1="2.79" y1="70.89" x2="2.79" y2="97.53" width="0.254" layer="21"/>
+<wire x1="2.79" y1="97.53" x2="15.6" y2="97.53" width="0.254" layer="21"/>
+<wire x1="15.6" y1="97.53" x2="15.6" y2="70.72" width="0.254" layer="21"/>
+<wire x1="15.6" y1="70.72" x2="2.8" y2="70.72" width="0.254" layer="21"/>
+<wire x1="2.8" y1="70.72" x2="2.8" y2="70.95" width="0.254" layer="21"/>
+<wire x1="76.78" y1="97.07" x2="93.54" y2="97.07" width="0.254" layer="21"/>
+<wire x1="93.54" y1="97.07" x2="93.54" y2="97.11" width="0.254" layer="21"/>
+<wire x1="77.93" y1="71.63" x2="93.02" y2="71.63" width="0.254" layer="21"/>
+<wire x1="93.02" y1="71.63" x2="93.02" y2="71.59" width="0.254" layer="21"/>
 </plain>
 <attributes>
@@
 <element name="CN4" library="con-phoenix-250" package="MCV4" value="MCV_05/4-G-2,5V" x="78.65" y="42.37" smashed="yes" rot="R270">
 <attribute name="NAME" x="83.55" y="39.71" size="1.778" layer="25" ratio="10" rot="R270"/>
-<attribute name="VALUE" x="72.281" y="46.66" size="1.778" layer="27" ratio="10" rot="R270"/>
 </element>
 <element name="CN5" library="con-molex" package="53047-04" value="53047-04" x="79.43" y="26.685" smashed="yes" rot="R90">
@@
 <attribute name="OC_FARNELL" value="9733060" x="79.43" y="26.685" size="1.778" layer="27" rot="R90" display="off"/>
 <attribute name="NAME" x="82.84" y="24.5" size="1.27" layer="25" rot="R90"/>
-<attribute name="VALUE" x="82.68" y="24.06" size="1.27" layer="27" rot="R90"/>
 </element>
 <element name="CN6" library="con-phoenix-250" package="MCV4" value="MCV_05/4-G-2,5V" x="34.29" y="95.105" smashed="yes">
@@
 <polygon width="0.3048" layer="16">
 <vertex x="-18.57" y="111.11"/>
-<vertex x="115.16" y="110.82"/>
+<vertex x="115.16" y="111.1"/>
 <vertex x="115.22" y="-11.54"/>
-<vertex x="-11.11" y="-11.13"/>
+<vertex x="-18.65" y="-11.13"/>
 <vertex x="-18.81" y="111.05"/>
 </polygon>
@@
 <wire x1="79.47" y1="64.22" x2="78.68" y2="65.91" width="0.4064" layer="1"/>
 <via x="78.68" y="65.91" extent="1-16" drill="0.6" shape="square"/>
-<wire x1="78.68" y1="65.91" x2="78.67" y2="69.54" width="0.4064" layer="16"/>
-<wire x1="78.67" y1="69.54" x2="75.29" y2="72.92" width="0.4064" layer="16"/>
-<wire x1="86.02" y1="64.21" x2="86.02" y2="62.73" width="0.254" layer="1"/>
-<wire x1="86.02" y1="62.73" x2="86.13" y2="62.4" width="0.254" layer="1"/>
-<via x="86.13" y="62.4" extent="1-16" drill="0.6" shape="square"/>
-<wire x1="86.13" y1="62.4" x2="86.12" y2="54.38" width="0.254" layer="16"/>
-<wire x1="86.12" y1="54.38" x2="90.68" y2="49.82" width="0.254" layer="16"/>
-<wire x1="90.68" y1="49.82" x2="95.23" y2="49.77" width="0.254" layer="16"/>
+<wire x1="78.68" y1="65.91" x2="78.67" y2="69.54" width="0.254" layer="16"/>
+<wire x1="78.67" y1="69.54" x2="75.29" y2="72.92" width="0.254" layer="16"/>
+<wire x1="86.02" y1="64.21" x2="86.02" y2="62.4" width="0.254" layer="1"/>
+<via x="86.02" y="62.4" extent="1-16" drill="0.6" shape="square"/>
+<wire x1="86.02" y1="62.4" x2="86.03" y2="54.38" width="0.254" layer="16"/>
+<wire x1="86.03" y1="54.38" x2="90.68" y2="49.76" width="0.254" layer="16"/>
+<wire x1="90.68" y1="49.76" x2="95.23" y2="49.77" width="0.254" layer="16"/>
 <wire x1="95.23" y1="49.77" x2="95.29" y2="49.76" width="0.254" layer="16"/>
 </signal>
@@
 <contactref element="CN25" pad="4"/>
 <contactref element="R4" pad="1"/>
-<wire x1="76.56" y1="68.79" x2="95.61" y2="87.84" width="0.254" layer="1"/>
-<wire x1="95.61" y1="87.84" x2="95.61" y2="88.16" width="0.254" layer="1"/>
+<wire x1="76.56" y1="68.79" x2="76.56" y2="69.11" width="0.254" layer="1"/>
+<wire x1="76.56" y1="69.11" x2="95.61" y2="88.16" width="0.254" layer="1"/>
 </signal>
 <signal name="N$12">
 <contactref element="SJ5" pad="1"/>
 <contactref element="CN25" pad="5"/>
-<wire x1="86.05" y1="69.44" x2="95.61" y2="85.62" width="0.254" layer="1"/>
+<wire x1="86.05" y1="69.44" x2="86.05" y2="76.06" width="0.254" layer="1"/>
+<wire x1="86.05" y1="76.06" x2="95.61" y2="85.62" width="0.254" layer="1"/>
 </signal>
 <signal name="CN2_5V">

Commit message: Revised Version 1
Parts:
- moved R2 0.12 mm to (59.0, 77.3)
Routing:
- net MW_SDA: track 96.6 -> 74.2 mm
- net VCC: track 319.8 -> 313.1 mm
- net N$11: track 27.3 -> 32.6 mm
- net N$12: track 20.1 -> 24.2 mm
- net V3_3: track 108.2 -> 111.3 mm
- net N$6: track 22.9 -> 24.5 mm
- net MW_TX0: track 53.3 -> 54.5 mm
- net N$7: track 4.54 -> 5.67 mm
- net MW_RX2: track 17.6 -> 18.6 mm
- net MW_RX1: track 15.9 -> 16.8 mm
Other:
- board text added: "Boiko, Chehadeh, Alansari, Alrheis, Ayyad"
- board text removed: "Boiko, Chehadeh, Alansari, Ayyad, Alrheis"
